Commit message: ackerman works

File: description/Traxxes.xacro (robot description, xacro)
@@ -1,8 +1,10 @@
 <?xml version="1.0"?>
 <robot xmlns:xacro="http://www.ros.org/wiki/xacro">
+  <xacro:include filename="inertial_macros.xacro" />
+  <!-- car geometry -->
   <xacro:arg name="wheel_diameter" default="0.112" />
   <xacro:property name="wheel_radius" value="${$(arg wheel_diameter)/2}" />
   <xacro:property name="wheel_width" value="0.047" />
-  <xacro:property name="wheel_friction" value="1.5" />
+  <xacro:property name="wheel_friction" value="1.0" />
   <xacro:property name="wheelbase_length" value="0.3429" />
   <xacro:property name="wheelbase_width" value="0.25" />
@@ -14,29 +16,17 @@
   <xacro:property name="chassis_elevation" value="-0.01" />
   <xacro:property name="chassis_mass" value="${total_mass-4*wheel_mass}" />
-  <xacro:include filename="inertial_macros.xacro" />
+  <!-- Steering params -->
+  <xacro:property name="steering_velocity" value="2.0" />
+  <xacro:property name="steering_upper_limit" value="1.0" />
+  <xacro:property name="steering_lower_limit" value="-1.0" />
+  <xacro:property name="steering_effort" value="2.0" />
   <!-- Base link -->
-  <link name="base_link">
-    <visual>
-      <geometry>
-        <cylinder length="0.01" radius="0.01" />
-      </geometry>
-      <material name="black">
-        <color rgba="0 0 0 1" />
-      </material>
-    </visual>
-    <collision>
-      <geometry>
-        <cylinder length="0.01" radius="0.01" />
-      </geometry>
-    </collision>
-    <xacro:inertial_cylinder mass="0.1" radius="0.01" length="0.01">
-      <origin xyz="0 0 0" rpy="0 0 0" />
-    </xacro:inertial_cylinder>
-  </link>
-  <!-- <joint name="base_link_joint" type="fixed">
+  <link name="base_link"></link>
+  <link name="base_footprint"></link>
+  <joint name="base_link_joint" type="fixed">
     <parent link="base_link" />
     <child link="base_footprint" />
     <origin rpy="0 0 0" xyz="0 0 0" />
-  </joint> -->
+  </joint>
   <!-- Chassis -->
   <link name="chassis_link">
@@ -130,5 +120,39 @@
     </xacro:inertial_cylinder>
   </link>
-  <link name="dummy_left">
+  <link name="front_left_wheel">
+    <visual>
+      <geometry>
+        <cylinder length="${wheel_width}" radius="${wheel_radius}" />
+      </geometry>
+      <material name="black">
+        <color rgba="0 0 0 1" />
+      </material>
+    </visual>
+    <collision>
+      <geometry>
+        <cylinder length="${wheel_width}" radius="${wheel_radius}" />
+      </geometry>
+    </collision>
+    <xacro:inertial_cylinder mass="${wheel_mass}" radius="${wheel_radius}" length="${wheel_width}">
+      <origin xyz="0 0 0" rpy="0 0 0" />
+    </xacro:inertial_cylinder>
+  </link>
+  <joint name="front_left_steer_joint" type="revolute">
+    <parent link="chassis_link" />
+    <child link="front_left_steer" />
+    <axis xyz="0 0 1" />
+    <origin rpy="0 0 0" xyz="${wheelbase_length/2} ${wheelbase_width/2} 0" />
+    <limit lower="${steering_lower_limit}" upper="${steering_upper_limit}"
+      effort="${steering_effort}" velocity="${steering_velocity}" />
+    <dynamics damping="0.0" friction="0.2" />
+  </joint>
+  <joint name="front_left_wheel_joint" type="continuous">
+    <parent link="front_left_steer" />
+    <child link="front_left_wheel" />
+    <axis xyz="0 0 1" />
+    <origin rpy="${-pi/2} 0 0" xyz="0 0 0" />
+  </joint>
+  <!-- front_right -->
+  <link name="front_right_steer">
     <visual>
       <geometry>
@@ -148,40 +172,57 @@
     </xacro:inertial_cylinder>
   </link>
-  <link name="front_left_wheel">
-    <visual>
-      <geometry>
-        <cylinder length="${wheel_width}" radius="${wheel_radius}" />
-      </geometry>
-      <material name="black">
-        <color rgba="0 0 0 1" />
-      </material>
-    </visual>
-    <collision>
-      <geometry>
-        <cylinder length="${wheel_width}" radius="${wheel_radius}" />
-      </geometry>
-    </collision>
-    <xacro:inertial_cylinder mass="${wheel_mass}" radius="${wheel_radius}" length="${wheel_width}">
-      <origin xyz="0 0 0" rpy="0 0 0" />
-    </xacro:inertial_cylinder>
-  </link>
-  <joint name="front_left_steer_joint" type="revolute">
-    <parent link="chassis_link" />
-    <child link="front_left_steer" />
-    <axis xyz="0 0 1" />
-    <origin rpy="0 0 0" xyz="${wheelbase_length/2} ${wheelbase_width/2} 0" />
-    <limit lower="-0.7" upper="0.7" effort="0.5" velocity="1.0" />
-    <!-- <dynamics damping="0.0" friction="0.2"/> -->
-  </joint>
-  <joint name="dummy_left_joint" type="fixed">
-    <parent link="front_left_steer" />
-    <child link="dummy_left" />
-    <origin rpy="0 0 0" xyz="0 0 0" />
-  </joint>
-  <joint name="front_left_wheel_joint" type="continuous">
-    <parent link="dummy_left" />
-    <child link="front_left_wheel" />
+  <link name="front_right_wheel">
+    <visual>
+      <geometry>
+        <cylinder length="${wheel_width}" radius="${wheel_radius}" />
+      </geometry>
+      <material name="black">
+        <color rgba="0 0 0 1" />
+      </material>
+    </visual>
+    <collision>
+      <geometry>
+        <cylinder length="${wheel_width}" radius="${wheel_radius}" />
+      </geometry>
+    </collision>
+    <xacro:inertial_cylinder mass="${wheel_mass}" radius="${wheel_radius}" length="${wheel_width}">
+      <origin xyz="0 0 0" rpy="0 0 0" />
+    </xacro:inertial_cylinder>
+  </link>
+  <joint name="front_right_steer_joint" type="revolute">
+    <parent link="chassis_link" />
+    <child link="front_right_steer" />
+    <axis xyz="0 0 1" />
+    <origin rpy="0 0 0" xyz="${wheelbase_length/2} -${wheelbase_width/2} 0" />
+    <limit lower="${steering_lower_limit}" upper="${steering_upper_limit}"
+      effort="${steering_effort}" velocity="${steering_velocity}" />
+    <dynamics damping="0.0" friction="0.2" />
+  </joint>
+  <joint name="front_right_right_joint" type="continuous">
+    <parent link="front_right_steer" />
+    <child link="front_right_wheel" />
     <axis xyz="0 0 1" />
     <origin rpy="${-pi/2} 0 0" xyz="0 0 0" />
   </joint>
+  <!-- Gazebo interface -->
+  <gazebo reference="front_left_wheel">
+    <mu1 value="${wheel_friction}" />
+    <mu2 value="${wheel_friction}" />
+    <material>Gazebo/DarkGrey</material>
+  </gazebo>
+  <gazebo reference="front_right_wheel">
+    <mu1 value="${wheel_friction}" />
+    <mu2 value="${wheel_friction}" />
+    <material>Gazebo/DarkGrey</material>
+  </gazebo>
+  <gazebo reference="back_left_wheel">
+    <mu1 value="${wheel_friction}" />
+    <mu2 value="${wheel_friction}" />
+    <material>Gazebo/DarkGrey</material>
+  </gazebo>
+  <gazebo reference="back_right_wheel">
+    <mu1 value="${wheel_friction}" />
+    <mu2 value="${wheel_friction}" />
+    <material>Gazebo/DarkGrey</material>
+  </gazebo>
 </robot>

File: description/ros2_control.xacro (robot description, xacro)
@@ -91,5 +91,5 @@
             <state_interface name="position"/>
         </joint>
-        <joint name="front_right_wheel_steer_joint">
+        <joint name="front_right_steer_joint">
             <command_interface name="position">
                 <param name="min">-1</param>
@@ -99,5 +99,5 @@
             <state_interface name="position"/>
         </joint>
-        <joint name="front_left_wheel_steer_joint">
+        <joint name="front_left_steer_joint">
             <command_interface name="position">
                 <param name="min">-1</param>

Commit message: odom works!

File: description/Traxxes.xacro (robot description, xacro)
@@ -22,7 +22,41 @@
   <xacro:property name="steering_effort" value="2.0" />
   <!-- Base link -->
-  <link name="base_link"></link>
-  <link name="base_footprint"></link>
-  <joint name="base_link_joint" type="fixed">
+  <link name="base_link">
+    <visual>
+      <geometry>
+        <cylinder length="0.001" radius="0.001" />
+      </geometry>
+      <material name="black">
+        <color rgba="0 0 0 1" />
+      </material>
+    </visual>
+    <collision>
+      <geometry>
+        <cylinder length="0.01" radius="0.01" />
+      </geometry>
+    </collision>
+    <xacro:inertial_cylinder mass="0.001" radius="0.001" length="0.001">
+      <origin xyz="0 0 0" rpy="0 0 0" />
+    </xacro:inertial_cylinder>
+  </link>
+  <link name="base_footprint">
+    <visual>
+      <geometry>
+        <cylinder length="0.001" radius="0.001" />
+      </geometry>
+      <material name="black">
+        <color rgba="0 0 0 1" />
+      </material>
+    </visual>
+    <collision>
+      <geometry>
+        <cylinder length="0.01" radius="0.01" />
+      </geometry>
+    </collision>
+    <xacro:inertial_cylinder mass="0.001" radius="0.001" length="0.001">
+      <origin xyz="0 0 0" rpy="0 0 0" />
+    </xacro:inertial_cylinder>
+  </link>
+  <joint name="base_footprint_joint" type="fixed">
     <parent link="base_link" />
     <child link="base_footprint" />

File: description/lidar.xacro (robot description, xacro)
@@ -1,30 +1,30 @@
 <?xml version="1.0"?>
-<robot xmlns:xacro="http://www.ros.org/wiki/xacro" >
+<robot xmlns:xacro="http://www.ros.org/wiki/xacro">
     <joint name="laser_joint" type="fixed">
-        <parent link="chassis"/>
-        <child link="laser_frame"/>
-        <origin xyz="0.122 0 0.212" rpy="0 0 0"/>
+        <parent link="chassis_link" />
+        <child link="laser_frame" />
+        <origin xyz="0.122 0 0.1" rpy="0 0 0" />
     </joint>
     <link name="laser_frame">
         <visual>
             <geometry>
-                <cylinder radius="0.05" length="0.04"/>
+                <cylinder radius="0.05" length="0.04" />
             </geometry>
-            <material name="black"/>
+            <material name="black" />
         </visual>
         <visual>
-            <origin xyz="0 0 -0.05"/>
+            <origin xyz="0 0 -0.05" />
             <geometry>
-                <cylinder radius="0.01" length="0.1"/>
+                <cylinder radius="0.01" length="0.1" />
             </geometry>
-            <material name="black"/>
+            <material name="black" />
         </visual>
         <collision>
             <geometry>
-                <cylinder radius="0.05" length="0.04"/>
+                <cylinder radius="0.05" length="0.04" />
             </geometry>
         </collision>
         <xacro:inertial_cylinder mass="0.1" length="0.04" radius="0.05">
-            <origin xyz="0 0 0" rpy="0 0 0"/>
+            <origin xyz="0 0 0" rpy="0 0 0" />
         </xacro:inertial_cylinder>
     </link>
@@ -34,5 +34,5 @@
             <pose> 0 0 0 0 0 0 </pose>
             <visualize>false</visualize>
-            <update_rate>10</update_rate>
+            <update_rate>5</update_rate>
             <ray>
                 <scan>
@@ -45,5 +45,5 @@
                 <range>
                     <min>0.3</min>
-                    <max>12</max>
+                    <max>7</max>
                 </range>
             </ray>

File: description/robot.urdf.xacro (robot description, xacro)
@@ -1,11 +1,8 @@
 <?xml version="1.0"?>
 <robot xmlns:xacro="http://www.ros.org/wiki/xacro"  name="robot">
-    <!-- <xacro:arg name="use_ros2_control" default="true"/>
-    <xacro:arg name="sim_mode" default="true"/> -->
+    <xacro:arg name="use_ros2_control" default="true"/>
+    <xacro:arg name="sim_mode" default="true"/>
     <xacro:include filename="Traxxes.xacro" />
     <xacro:include filename="ros2_control.xacro" />
-    <!-- <xacro:unless value="$(arg use_ros2_control)">
-        <xacro:include filename="gazebo_control.xacro" />
-    </xacro:unless> -->
     <!-- <xacro:include filename="lidar.xacro" /> -->
     <!-- <xacro:include filename="camera.xacro" /> -->

File: description/ros2_control.xacro (robot description, xacro)
@@ -1,74 +1,4 @@
 <?xml version="1.0"?>
 <robot xmlns:xacro="http://www.ros.org/wiki/xacro">
-    <!-- <xacro:unless value="$(arg sim_mode)">
-        <ros2_control name="RealRobot" type="system">
-            <hardware>
-                <plugin>diffdrive_arduino/DiffDriveArduino</plugin>
-                <param name="left_wheel_name">left_wheel_joint</param>
-                <param name="right_wheel_name">right_wheel_joint</param>
-                <param name="loop_rate">30</param>
-                <param name="device">/dev/ttyUSB0</param>
-                <param name="baud_rate">57600</param>
-                <param name="timeout">1000</param>
-                <param name="enc_counts_per_rev">3436</param>
-            </hardware>
-            <joint name="left_wheel_joint">
-                <command_interface name="velocity">
-                    <param name="min">-10</param>
-                    <param name="max">10</param>
-                </command_interface>
-                <state_interface name="velocity"/>
-                <state_interface name="position"/>
-            </joint>
-            <joint name="right_wheel_joint">
-                <command_interface name="velocity">
-                    <param name="min">-10</param>
-                    <param name="max">10</param>
-                </command_interface>
-                <state_interface name="velocity"/>
-                <state_interface name="position"/>
-            </joint>
-        </ros2_control>
-    </xacro:unless> -->
-    <!-- <xacro:if value="$(arg sim_mode)">
-        <ros2_control name="GazeboSystem" type="system">
-            <hardware>
-                <plugin>gazebo_ros2_control/GazeboSystem</plugin>
-            </hardware>
-            <joint name="left_wheel_joint">
-                <command_interface name="velocity">
-                    <param name="min">-10</param>
-                    <param name="max">10</param>
-                </command_interface>
-                <state_interface name="velocity"/>
-                <state_interface name="position"/>
-            </joint>
-            <joint name="right_wheel_joint">
-                <command_interface name="velocity">
-                    <param name="min">-10</param>
-                    <param name="max">10</param>
-                </command_interface>
-                <state_interface name="velocity"/>
-                <state_interface name="position"/>
-            </joint>
-        </ros2_control>
-    </xacro:if>  -->
-    <!-- <gazebo>
-        <plugin name="gazebo_ros2_control" filename="libgazebo_ros2_control.so">
-            <parameters>$(find rc_car)/config/my_controllers.yaml</parameters>
-            <parameters>$(find rc_car)/config/gaz_ros2_ctl_use_sim.yaml</parameters>
-        </plugin>
-    </gazebo> -->
-<!--
-    <plugin name="joint_broad" filename="libgazebo_ros_joint_state_publisher.so">
-        <ros>
-            <remapping>~/out:=joint_states</remapping>
-        </ros>
-        <update_rate>30</update_rate>
-        <joint_name>front_left_steering_joint</joint_name>
-        <joint_name>front_right_steering_joint</joint_name>
-        <joint_name>rear_left_wheel_joint</joint_name>
-        <joint_name>rear_right_wheel_joint</joint_name>
-    </plugin> -->
     <ros2_control name="GazeboSystem" type="system">
         <hardware>
@@ -80,6 +10,6 @@
                 <param name="max">10</param>
             </command_interface>
-            <state_interface name="velocity"/>
-            <state_interface name="position"/>
+            <state_interface name="velocity" />
+            <state_interface name="position" />
         </joint>
         <joint name="back_left_wheel_joint">
@@ -88,6 +18,6 @@
                 <param name="max">10</param>
             </command_interface>
-            <state_interface name="velocity"/>
-            <state_interface name="position"/>
+            <state_interface name="velocity" />
+            <state_interface name="position" />
         </joint>
         <joint name="front_right_steer_joint">
@@ -97,5 +27,5 @@
             </command_interface>
             <!-- <state_interface name="velocity"/>  -->
-            <state_interface name="position"/>
+            <state_interface name="position" />
         </joint>
         <joint name="front_left_steer_joint">
@@ -105,5 +35,5 @@
             </command_interface>
             <!-- <state_interface name="velocity"/>  -->
-            <state_interface name="position"/>
+            <state_interface name="position" />
         </joint>
     </ros2_control>
