Commit message: odom works

File: description/Traxxes.xacro (robot description, xacro)
@@ -6,7 +6,7 @@
   <xacro:property name="wheel_radius" value="${$(arg wheel_diameter)/2}" />
   <xacro:property name="wheel_width" value="0.047" />
-  <xacro:property name="wheel_friction" value="1.0" />
-  <xacro:property name="wheelbase_length" value="0.3429" />
-  <xacro:property name="wheelbase_width" value="0.25" />
+  <xacro:property name="wheel_friction" value="0.8" />
+  <xacro:property name="wheelbase" value="0.3429" />
+  <xacro:property name="track_width" value="0.25" />
   <xacro:property name="chassis_width" value="0.18" />
   <xacro:property name="wheel_mass" value="0.1" />
@@ -17,11 +17,11 @@
   <xacro:property name="chassis_mass" value="${total_mass-4*wheel_mass}" />
   <!-- Steering params -->
-  <xacro:property name="steering_velocity" value="2.0" />
-  <xacro:property name="steering_upper_limit" value="1.0" />
-  <xacro:property name="steering_lower_limit" value="-1.0" />
-  <xacro:property name="steering_effort" value="2.0" />
+  <xacro:property name="steering_velocity" value="1.0" />
+  <xacro:property name="steering_upper_limit" value="0.7" />
+  <xacro:property name="steering_lower_limit" value="-0.7" />
+  <xacro:property name="steering_effort" value="1000.0" />
   <!-- Base link -->
   <link name="base_link">
-    <visual>
+   <visual>
       <geometry>
         <cylinder length="0.001" radius="0.001" />
@@ -40,5 +40,5 @@
     </xacro:inertial_cylinder>
   </link>
-  <link name="base_footprint">
+  <!-- <link name="base_footprint">
     <visual>
       <geometry>
@@ -62,19 +62,18 @@
     <child link="base_footprint" />
     <origin rpy="0 0 0" xyz="0 0 0" />
-  </joint>
+  </joint> -->
   <!-- Chassis -->
   <link name="chassis_link">
     <visual>
       <geometry>
-        <box size="${wheelbase_length} ${chassis_width} ${chassis_height}" />
-      </geometry>
-    </visual>
-    <collision>
-      <geometry>
-        <box size="${wheelbase_length} ${chassis_width} ${chassis_height}" />
-      </geometry>
-    </collision>
-    <xacro:inertial_box mass="${chassis_mass}" x="${wheelbase_length}" y="${chassis_width}"
-      z="${chassis_height}">
+        <box size="${wheelbase} ${chassis_width} ${chassis_height}" />
+      </geometry>
+    </visual>
+    <collision>
+      <geometry>
+        <box size="${wheelbase} ${chassis_width} ${chassis_height}" />
+      </geometry>
+    </collision>
+    <xacro:inertial_box mass="${chassis_mass}" x="${wheelbase}" y="${chassis_width}" z="${chassis_height}">
       <origin xyz="0 0 0" rpy="0 0 0" />
     </xacro:inertial_box>
@@ -83,5 +82,6 @@
     <parent link="base_link" />
     <child link="chassis_link" />
-    <origin rpy="0 0 0" xyz="${wheelbase_length/2} 0 ${chassis_height/2 + chassis_elevation}" />
+    <!-- <origin rpy="0 0 0" xyz="${wheelbase/2} 0 ${chassis_height/2 + chassis_elevation}" /> -->
+    <origin rpy="0 0 0" xyz="0 0 ${chassis_height/2 + chassis_elevation}" />
   </joint>
   <!-- Rear Left wheel -->
@@ -108,5 +108,5 @@
     <child link="back_left_wheel" />
     <axis xyz="0 0 1" />
-    <origin rpy="${-pi/2} 0 0" xyz="-${wheelbase_length/2} ${wheelbase_width/2} 0" />
+    <origin rpy="${-pi/2} 0 0" xyz="-${wheelbase/2} ${track_width/2} 0" />
   </joint>
   <!-- Rear right wheel -->
@@ -133,5 +133,5 @@
     <child link="back_right_wheel" />
     <axis xyz="0 0 -1" />
-    <origin rpy="${-pi/2} 0 0" xyz="-${wheelbase_length/2} -${wheelbase_width/2} 0" />
+    <origin rpy="${pi/2} 0 0" xyz="-${wheelbase/2} -${track_width/2} 0" />
   </joint>
   <!-- front_left_ -->
@@ -176,7 +176,6 @@
     <child link="front_left_steer" />
     <axis xyz="0 0 1" />
-    <origin rpy="0 0 0" xyz="${wheelbase_length/2} ${wheelbase_width/2} 0" />
-    <limit lower="${steering_lower_limit}" upper="${steering_upper_limit}"
-      effort="${steering_effort}" velocity="${steering_velocity}" />
+    <origin rpy="0 0 0" xyz="${wheelbase/2} ${track_width/2} 0" />
+    <limit lower="${steering_lower_limit}" upper="${steering_upper_limit}" effort="${steering_effort}" velocity="${steering_velocity}" />
     <dynamics damping="0.0" friction="0.2" />
   </joint>
@@ -228,14 +227,13 @@
     <child link="front_right_steer" />
     <axis xyz="0 0 1" />
-    <origin rpy="0 0 0" xyz="${wheelbase_length/2} -${wheelbase_width/2} 0" />
-    <limit lower="${steering_lower_limit}" upper="${steering_upper_limit}"
-      effort="${steering_effort}" velocity="${steering_velocity}" />
+    <origin rpy="0 0 0" xyz="${wheelbase/2} -${track_width/2} 0" />
+    <limit lower="${steering_lower_limit}" upper="${steering_upper_limit}" effort="${steering_effort}" velocity="${steering_velocity}" />
     <dynamics damping="0.0" friction="0.2" />
   </joint>
-  <joint name="front_right_right_joint" type="continuous">
+  <joint name="front_right_wheel_joint" type="continuous">
     <parent link="front_right_steer" />
     <child link="front_right_wheel" />
-    <axis xyz="0 0 1" />
-    <origin rpy="${-pi/2} 0 0" xyz="0 0 0" />
+    <axis xyz="0 0 -1" />
+    <origin rpy="${pi/2} 0 0" xyz="0 0 0" />
   </joint>
   <!-- Gazebo interface -->

File: description/ros2_control.xacro (robot description, xacro)
@@ -1,4 +1,6 @@
 <?xml version="1.0"?>
 <robot xmlns:xacro="http://www.ros.org/wiki/xacro">
+    <xacro:property name="steering_upper_limit" value="0.7" />
+    <xacro:property name="steering_lower_limit" value="-0.7" />
     <ros2_control name="GazeboSystem" type="system">
         <hardware>
@@ -7,6 +9,6 @@
         <joint name="back_right_wheel_joint">
             <command_interface name="velocity">
-                <param name="min">-10</param>
-                <param name="max">10</param>
+                <param name="min">-1</param>
+                <param name="max">1</param>
             </command_interface>
             <state_interface name="velocity" />
@@ -15,6 +17,6 @@
         <joint name="back_left_wheel_joint">
             <command_interface name="velocity">
-                <param name="min">-10</param>
-                <param name="max">10</param>
+                <param name="min">-1</param>
+                <param name="max">1</param>
             </command_interface>
             <state_interface name="velocity" />
@@ -23,6 +25,6 @@
         <joint name="front_right_steer_joint">
             <command_interface name="position">
-                <param name="min">-1</param>
-                <param name="max">1</param>
+                <param name="min">"${steering_lower_limit}"</param>
+                <param name="max">"${steering_upper_limit}"</param>
             </command_interface>
             <!-- <state_interface name="velocity"/>  -->
@@ -31,6 +33,6 @@
         <joint name="front_left_steer_joint">
             <command_interface name="position">
-                <param name="min">-1</param>
-                <param name="max">1</param>
+                <param name="min">"${steering_lower_limit}"</param>
+                <param name="max">"${steering_upper_limit}"</param>
             </command_interface>
             <!-- <state_interface name="velocity"/>  -->
