Commit message: add lidar and camera

File: rc_car/description/camera.xacro (robot description, xacro)
@@ -2,7 +2,7 @@
 <robot xmlns:xacro="http://www.ros.org/wiki/xacro" >
     <joint name="camera_joint" type="fixed">
-        <parent link="chassis"/>
+        <parent link="chassis_link"/>
         <child link="camera_link"/>
-        <origin xyz="0.276 0 0.181" rpy="0 0.18 0"/>
+        <origin xyz="0.15 0 0.1" rpy="0 0.18 0"/>
     </joint>
     <link name="camera_link">

File: rc_car/description/lidar.xacro (robot description, xacro)
@@ -4,5 +4,5 @@
         <parent link="chassis_link" />
         <child link="laser_frame" />
-        <origin xyz="0.122 0 0.1" rpy="0 0 0" />
+        <origin xyz="-0.12 0 0.10" rpy="0 0 0" />
     </joint>
     <link name="laser_frame">
@@ -33,5 +33,5 @@
         <sensor name="laser" type="ray">
             <pose> 0 0 0 0 0 0 </pose>
-            <visualize>false</visualize>
+            <visualize>true</visualize>
             <update_rate>5</update_rate>
             <ray>

File: rc_car/description/robot.urdf.xacro (robot description, xacro)
@@ -5,6 +5,6 @@
     <xacro:include filename="Traxxes.xacro" />
     <xacro:include filename="ros2_control.xacro" />
-    <!-- <xacro:include filename="lidar.xacro" /> -->
-    <!-- <xacro:include filename="camera.xacro" /> -->
+    <xacro:include filename="lidar.xacro" />
+    <xacro:include filename="camera.xacro" />
     <!-- <xacro:include filename="depth_camera.xacro" /> -->
     <!-- <xacro:include filename="face.xacro" /> -->
