Commit message: slam works

File: rc_car/description/Traxxes.xacro (robot description, xacro)
@@ -40,5 +40,5 @@
     </xacro:inertial_cylinder>
   </link>
-  <!-- <link name="base_footprint">
+  <link name="base_footprint">
     <visual>
       <geometry>
@@ -62,5 +62,5 @@
     <child link="base_footprint" />
     <origin rpy="0 0 0" xyz="0 0 0" />
-  </joint> -->
+  </joint>
   <!-- Chassis -->
   <link name="chassis_link">

Commit message: add realrobot

File: rc_car/description/Traxxes.xacro (robot description, xacro)
@@ -97,4 +97,5 @@
     <collision>
       <geometry>
+        <!-- <sphere radius="${wheel_radius}" /> -->
         <cylinder length="${wheel_width}" radius="${wheel_radius}" />
       </geometry>

File: rc_car/description/robot.urdf.xacro (robot description, xacro)
@@ -2,7 +2,11 @@
 <robot xmlns:xacro="http://www.ros.org/wiki/xacro"  name="robot">
     <xacro:arg name="use_ros2_control" default="true"/>
-    <xacro:arg name="sim_mode" default="true"/>
+    <xacro:arg name="sim_mode" default="false"/>
     <xacro:include filename="Traxxes.xacro" />
-    <xacro:include filename="ros2_control.xacro" />
+    <xacro:if value="$(arg use_ros2_control)">
+        <xacro:include filename="ros2_control.xacro" />
+    </xacro:if>
+    <!-- <xacro:unless value="$(arg use_ros2_control)">
+    </xacro:unless> -->
     <xacro:include filename="lidar.xacro" />
     <xacro:include filename="camera.xacro" />

File: rc_car/description/ros2_control.xacro (robot description, xacro)
@@ -3,42 +3,93 @@
     <xacro:property name="steering_upper_limit" value="0.7" />
     <xacro:property name="steering_lower_limit" value="-0.7" />
-    <ros2_control name="GazeboSystem" type="system">
-        <hardware>
-            <plugin>gazebo_ros2_control/GazeboSystem</plugin>
-        </hardware>
-        <joint name="back_right_wheel_joint">
-            <command_interface name="velocity">
-                <param name="min">-1</param>
-                <param name="max">1</param>
-            </command_interface>
-            <state_interface name="velocity" />
-            <state_interface name="position" />
-        </joint>
-        <joint name="back_left_wheel_joint">
-            <command_interface name="velocity">
-                <param name="min">-1</param>
-                <param name="max">1</param>
-            </command_interface>
-            <state_interface name="velocity" />
-            <state_interface name="position" />
-        </joint>
-        <joint name="front_right_steer_joint">
-            <command_interface name="position">
-                <param name="min">"${steering_lower_limit}"</param>
-                <param name="max">"${steering_upper_limit}"</param>
-            </command_interface>
-            <!-- <state_interface name="velocity"/>  -->
-            <state_interface name="position" />
-        </joint>
-        <joint name="front_left_steer_joint">
-            <command_interface name="position">
-                <param name="min">"${steering_lower_limit}"</param>
-                <param name="max">"${steering_upper_limit}"</param>
-            </command_interface>
-            <!-- <state_interface name="velocity"/>  -->
-            <state_interface name="position" />
-        </joint>
-    </ros2_control>
+    <xacro:unless value="$(arg sim_mode)">
+        <ros2_control name="RealRobot" type="system">
+            <hardware>
+                <!-- this pluging tells the program how to tack to the simulation -->
+                <plugin>diffdrive_arduino/DiffDriveArduino</plugin>
+                <param name="left_wheel_name">back_right_wheel_joint</param>
+                <param name="right_wheel_name">front_left_steer_joint</param>
+                <param name="loop_rate">30</param>
+                <param name="device">/dev/ttyACM0</param>
+                <param name="baud_rate">57600</param>
+                <param name="timeout">1000</param>
+                <param name="enc_counts_per_rev">3450</param>
+            </hardware>
+            <joint name="back_right_wheel_joint">
+                <command_interface name="velocity">
+                    <param name="min">-1</param>
+                    <param name="max">1</param>
+                </command_interface>
+                <state_interface name="velocity" />
+                <state_interface name="position" />
+            </joint>
+            <joint name="back_left_wheel_joint">
+                <command_interface name="velocity">
+                    <param name="min">-1</param>
+                    <param name="max">1</param>
+                </command_interface>
+                <state_interface name="velocity" />
+                <state_interface name="position" />
+            </joint>
+            <joint name="front_right_steer_joint">
+                <command_interface name="position">
+                    <param name="min">"${steering_lower_limit}"</param>
+                    <param name="max">"${steering_upper_limit}"</param>
+                </command_interface>
+                <!-- <state_interface name="velocity"/>  -->
+                <state_interface name="position" />
+            </joint>
+            <joint name="front_left_steer_joint">
+                <command_interface name="position">
+                    <param name="min">"${steering_lower_limit}"</param>
+                    <param name="max">"${steering_upper_limit}"</param>
+                </command_interface>
+                <!-- <state_interface name="velocity"/>  -->
+                <state_interface name="position" />
+            </joint>
+        </ros2_control>
+    </xacro:unless>
+    <xacro:if value="$(arg sim_mode)">
+        <ros2_control name="GazeboSystem" type="system">
+            <hardware>
+                <!-- this pluging tells the program how to tack to the simulation -->
+                <plugin>gazebo_ros2_control/GazeboSystem</plugin>
+            </hardware>
+            <joint name="back_right_wheel_joint">
+                <command_interface name="velocity">
+                    <param name="min">-1</param>
+                    <param name="max">1</param>
+                </command_interface>
+                <state_interface name="velocity" />
+                <state_interface name="position" />
+            </joint>
+            <joint name="back_left_wheel_joint">
+                <command_interface name="velocity">
+                    <param name="min">-1</param>
+                    <param name="max">1</param>
+                </command_interface>
+                <state_interface name="velocity" />
+                <state_interface name="position" />
+            </joint>
+            <joint name="front_right_steer_joint">
+                <command_interface name="position">
+                    <param name="min">"${steering_lower_limit}"</param>
+                    <param name="max">"${steering_upper_limit}"</param>
+                </command_interface>
+                <!-- <state_interface name="velocity"/>  -->
+                <state_interface name="position" />
+            </joint>
+            <joint name="front_left_steer_joint">
+                <command_interface name="position">
+                    <param name="min">"${steering_lower_limit}"</param>
+                    <param name="max">"${steering_upper_limit}"</param>
+                </command_interface>
+                <!-- <state_interface name="velocity"/>  -->
+                <state_interface name="position" />
+            </joint>
+        </ros2_control>
+    </xacro:if>
     <gazebo>
+        <!-- this gazebo pugin telles gazebo to use ros2_control -->
         <plugin name="gazebo_ros2_control" filename="libgazebo_ros2_control.so">
             <parameters>$(find rc_car)/config/ackermann_steering_controller.yaml</parameters>
