Commit message: change to bicycle model

File: rc_car/description/robot.urdf.xacro (robot description, xacro)
@@ -3,11 +3,6 @@
     <xacro:arg name="use_ros2_control" default="true"/>
     <xacro:arg name="sim_mode" default="false"/>
-    <xacro:include filename="Traxxes.xacro" />
-    <!-- we only use ros2_control, we don't use gazebo control -->
-    <xacro:if value="$(arg use_ros2_control)">
-        <xacro:include filename="ros2_control.xacro" />
-    </xacro:if>
-    <!-- <xacro:unless value="$(arg use_ros2_control)">
-    </xacro:unless> -->
+    <xacro:include filename="Traxxes_2DOF.xacro" />
+    <xacro:include filename="ros2_control_bicycle.xacro" />
     <xacro:include filename="lidar.xacro" />
     <xacro:include filename="camera.xacro" />
@@ -15,3 +10,7 @@
     <!-- <xacro:include filename="depth_camera.xacro" /> -->
     <!-- <xacro:include filename="face.xacro" /> -->
+    <!-- <xacro:if value="$(arg use_ros2_control)"> -->
+    <!-- </xacro:if>  -->
+    <!-- <xacro:unless value="$(arg use_ros2_control)">
+    </xacro:unless> -->
 </robot>

File: rc_car/description/ros2_control_bicycle.xacro (robot description, xacro)
@@ -1,4 +1,6 @@
 <?xml version="1.0"?>
 <robot xmlns:xacro="http://www.ros.org/wiki/xacro">
+    <!-- this file contains the hardware interface for ROS2_CONTROL -->
+    <!-- to expose the interfaces to resourse manager (in the controller manager) -->
     <xacro:property name="steering_upper_limit" value="0.7" />
     <xacro:property name="steering_lower_limit" value="-0.7" />
@@ -53,8 +55,16 @@
         <ros2_control name="GazeboSystem" type="system">
             <hardware>
-                <!-- this pluging tells the program how to tack to the simulation -->
+                <!-- this pluging tells the program how to talk to the simulation -->
                 <plugin>gazebo_ros2_control/GazeboSystem</plugin>
             </hardware>
-            <joint name="back_right_wheel_joint">
+            <joint name="back_central_wheel_joint">
+                <command_interface name="velocity">
+                    <param name="min">-10</param>
+                    <param name="max">10</param>
+                </command_interface>
+                <state_interface name="position" />
+                <state_interface name="velocity" />
+            </joint>
+            <!-- <joint name="back_left_wheel_joint">
                 <command_interface name="velocity">
                     <param name="min">-1</param>
@@ -63,29 +73,19 @@
                 <state_interface name="velocity" />
                 <state_interface name="position" />
-            </joint>
-            <joint name="back_left_wheel_joint">
-                <command_interface name="velocity">
-                    <param name="min">-1</param>
-                    <param name="max">1</param>
-                </command_interface>
-                <state_interface name="velocity" />
-                <state_interface name="position" />
-            </joint>
-            <joint name="front_right_steer_joint">
+            </joint> -->
+            <joint name="front_central_steer_joint">
                 <command_interface name="position">
                     <param name="min">"${steering_lower_limit}"</param>
                     <param name="max">"${steering_upper_limit}"</param>
                 </command_interface>
-                <!-- <state_interface name="velocity"/>  -->
                 <state_interface name="position" />
             </joint>
-            <joint name="front_left_steer_joint">
+            <!-- <joint name="front_left_steer_joint">
                 <command_interface name="position">
                     <param name="min">"${steering_lower_limit}"</param>
                     <param name="max">"${steering_upper_limit}"</param>
                 </command_interface>
-                <!-- <state_interface name="velocity"/>  -->
                 <state_interface name="position" />
-            </joint>
+            </joint> -->
         </ros2_control>
     </xacro:if>
@@ -93,5 +93,5 @@
         <!-- this gazebo pugin telles gazebo to use ros2_control -->
         <plugin name="gazebo_ros2_control" filename="libgazebo_ros2_control.so">
-            <parameters>$(find rc_car)/config/ackermann_steering_controller.yaml</parameters>
+            <parameters>$(find rc_car)/config/bicycle_steering_controller.yaml</parameters>
             <parameters>$(find rc_car)/config/gaz_ros2_ctl_use_sim.yaml</parameters>
         </plugin>

Commit message: edit robot launch

File: rc_car/description/robot.urdf.xacro (robot description, xacro)
@@ -6,7 +6,9 @@
     <xacro:include filename="ros2_control_bicycle.xacro" />
     <xacro:include filename="lidar.xacro" />
-    <xacro:include filename="camera.xacro" />
-    <xacro:include filename="imu.xacro"/>
-    <xacro:include filename="ground_truth.xacro"/>
+    <xacro:if value="$(arg sim_mode)">
+        <xacro:include filename="camera.xacro" />
+        <xacro:include filename="imu.xacro"/>
+        <xacro:include filename="ground_truth.xacro"/>
+    </xacro:if>
     <!-- <xacro:include filename="depth_camera.xacro" /> -->
     <!-- <xacro:include filename="face.xacro" /> -->

File: rc_car/description/ros2_control_bicycle.xacro (robot description, xacro)
@@ -9,44 +9,28 @@
             <hardware>
                 <!-- this pluging tells the program how to talk interface -->
-                <plugin>diffdrive_arduino/DiffDriveArduino</plugin>
-                <param name="left_wheel_name">back_right_wheel_joint</param>
-                <param name="right_wheel_name">front_left_steer_joint</param>
+                <plugin>diffdrive_arduino/DiffDriveArduinoHardware</plugin>
+                <param name="rear_wheel_name">back_central_wheel_joint</param>
+                <param name="front_wheel_name">front_central_steer_joint</param>
                 <param name="loop_rate">30</param>
                 <param name="device">/dev/ttyACM0</param>
                 <param name="baud_rate">57600</param>
-                <param name="timeout">1000</param>
+                <param name="timeout_ms">1000</param>
                 <param name="enc_counts_per_rev">3450</param>
             </hardware>
-            <joint name="back_right_wheel_joint">
+            <joint name="back_central_wheel_joint">
                 <command_interface name="velocity">
-                    <param name="min">-1</param>
-                    <param name="max">1</param>
+                    <param name="min">-10</param>
+                    <param name="max">10</param>
                 </command_interface>
-                <state_interface name="velocity" />
-                <state_interface name="position" />
+                <state_interface name="position"/>
+                <state_interface name="velocity"/>
             </joint>
-            <joint name="back_left_wheel_joint">
-                <command_interface name="velocity">
-                    <param name="min">-1</param>
-                    <param name="max">1</param>
-                </command_interface>
-                <state_interface name="velocity" />
-                <state_interface name="position" />
-            </joint>
-            <joint name="front_right_steer_joint">
+            <joint name="front_central_steer_joint">
                 <command_interface name="position">
                     <param name="min">"${steering_lower_limit}"</param>
                     <param name="max">"${steering_upper_limit}"</param>
                 </command_interface>
-                <!-- <state_interface name="velocity"/>  -->
-                <state_interface name="position" />
-            </joint>
-            <joint name="front_left_steer_joint">
-                <command_interface name="position">
-                    <param name="min">"${steering_lower_limit}"</param>
-                    <param name="max">"${steering_upper_limit}"</param>
-                </command_interface>
-                <!-- <state_interface name="velocity"/>  -->
-                <state_interface name="position" />
+                <state_interface name="position"/>
+                <state_interface name="velocity"/>
             </joint>
         </ros2_control>
@@ -66,12 +50,4 @@
                 <state_interface name="velocity" />
             </joint>
-            <!-- <joint name="back_left_wheel_joint">
-                <command_interface name="velocity">
-                    <param name="min">-1</param>
-                    <param name="max">1</param>
-                </command_interface>
-                <state_interface name="velocity" />
-                <state_interface name="position" />
-            </joint> -->
             <joint name="front_central_steer_joint">
                 <command_interface name="position">
@@ -81,11 +57,4 @@
                 <state_interface name="position" />
             </joint>
-            <!-- <joint name="front_left_steer_joint">
-                <command_interface name="position">
-                    <param name="min">"${steering_lower_limit}"</param>
-                    <param name="max">"${steering_upper_limit}"</param>
-                </command_interface>
-                <state_interface name="position" />
-            </joint> -->
         </ros2_control>
     </xacro:if>
