Commit message: fix simulation- show wheels in rviz

File: rc_car/description/Traxxes_2DOF.xacro (robot description, xacro)
@@ -238,5 +238,5 @@
     <child link="front_left_wheel" />
     <!-- <axis xyz="0 0 1" /> -->
-    <origin rpy="0 0 0" xyz="${wheelbase/2} ${track_width/2} 0" />
+    <origin rpy="${-pi/2} 0 0" xyz="${wheelbase/2} ${track_width/2} 0" />
   </joint>
   <!-- front_right -->
@@ -264,5 +264,5 @@
     <child link="front_right_wheel" />
     <!-- <axis xyz="0 0 -1" /> -->
-    <origin rpy="0 0 0" xyz="${wheelbase/2} -${track_width/2} 0" />
+    <origin rpy="${-pi/2} 0 0" xyz="${wheelbase/2} -${track_width/2} 0" />
   </joint>
   <!-- Gazebo interface -->

Commit message: rviz config

File: rc_car/description/Traxxes_2DOF.xacro (robot description, xacro)
@@ -18,6 +18,6 @@
   <!-- Steering params -->
   <xacro:property name="steering_velocity" value="0.2" />
-  <xacro:property name="steering_upper_limit" value="0.7" />
-  <xacro:property name="steering_lower_limit" value="-0.7" />
+  <xacro:property name="steering_upper_limit" value="0.6" />
+  <xacro:property name="steering_lower_limit" value="-0.6" />
   <xacro:property name="steering_effort" value="1000.0" />
   <!-- Base link -->

Commit message: amcl parameters: update resolution

File: rc_car/description/Traxxes_2DOF.xacro (robot description, xacro)
@@ -6,5 +6,5 @@
   <xacro:property name="wheel_radius" value="${$(arg wheel_diameter)/2}" />
   <xacro:property name="wheel_width" value="0.047" />
-  <xacro:property name="wheel_friction" value="0.8" />
+  <xacro:property name="wheel_friction" value="2.0" />
   <xacro:property name="wheelbase" value="0.3429" />
   <xacro:property name="track_width" value="0.25" />

Commit message: m

File: rc_car/description/Traxxes_2DOF.xacro (robot description, xacro)
@@ -7,5 +7,5 @@
   <xacro:property name="wheel_width" value="0.047" />
   <xacro:property name="wheel_friction" value="2.0" />
-  <xacro:property name="wheelbase" value="0.3429" />
+  <xacro:property name="wheelbase" value="0.335" />
   <xacro:property name="track_width" value="0.25" />
   <xacro:property name="chassis_width" value="0.18" />
