Commit message: update hardware files

File: src/rc_car/description/lidar.xacro (robot description, xacro)
@@ -4,5 +4,5 @@
         <parent link="chassis_link" />
         <child link="laser_frame" />
-        <origin xyz="-0.12 0 0.10" rpy="0 0 0" />
+        <origin xyz="-0.02 0 0.15" rpy="0 0 3.14159" />
     </joint>
     <link name="laser_frame">
